Commit message: changed config

File: husky_description/urdf/accessories/intel_realsense.urdf.xacro (robot description, xacro)
@@ -7,5 +7,5 @@
                min_range:=0.105          max_range:=8.0
                width:=640                height:=480
-               update_rate:=30
+               update_rate:=15
                robot_namespace:=/">
       <!-- this link is the origin for the camera's data -->
@@ -39,5 +39,5 @@
               <!-- give the color sensor a maximum range of 50m so that the simulation renders nicely -->
               <near>0.01</near>
-              <far>50.0</far>
+              <far>30.0</far>
             </clip>
           </camera>

File: husky_description/urdf/husky.urdf.xacro (robot description, xacro)
@@ -140,5 +140,5 @@
     <link name="realsense_mountpoint"/>
     <joint name="realsense_mountpoint_joint" type="fixed">
-      <origin xyz="0 0 0" rpy="0 0 -3.14159" />
+      <origin xyz="0 0 0" rpy="0 -0.2 -3.14159" />
       <parent link="$(arg realsense_mount)"/>
       <child link="realsense_mountpoint" />
